Commit message: integrated pipeline is added. fixed point cloud utils.

File: urdf/bed_0.urdf (robot description, URDF)
Before this commit: robot cube.urdf, 1 links, 0 joints
Links:
- link baseLink: geometry collision box size=0.6 1.7 0.4; visual box size=0.6 1.7 0.4

File: urdf/humanoid_with_rev.urdf (robot description, URDF)
Before this commit: robot dumpUrdf, 19 links, 18 joints
Joints:
- joint left_ankle: origin xyz=0.000000 -1.639480 0.000000 rpy=0 0 0 -> xyz=-0.3 -1.639480 0.000000 rpy=0 0 0
- joint right_ankle: origin xyz=0.000000 -1.639480 0.000000 rpy=0 0 0 -> xyz=-0.3 -1.639480 0.000000 rpy=0 0 0

Commit message: arm manipulation bugs are fixed. readme is added.

File: urdf/bed_0.urdf (robot description, URDF)
Before this commit: robot cube.urdf, 1 links, 0 joints
Links:
- link baseLink: geometry collision box size=0.6 1.5 0.4; visual box size=0.6 1.5 0.4

File: urdf/wiper.urdf (robot description, URDF)
Before this commit: robot wiper, 3 links, 2 joints
Links:
- link handle: geometry collision box size=0.04 0.04 0.04; visual box size=0.04 0.04 0.06
